File: ECU Outputs/ECUOutputs/ECUOutputs.sch (KiCad schematic (older format))
At the start: 13 parts, among them J4 ECU CONNECTOR, Q1 BSX46

Commit message: Updated manufacturer part numbers. Working on ECU outputs tester board.
Parts:
- removed Q1: BSX46, symbol Device:Q_NPN_CBE
- added Q1: BC817-40-TP, Package_TO_SOT_SMD:SOT-23, symbol Device:Q_NPN_BEC
- D1, D2, D3: value D -> MMSD4148T1G; footprint (none) -> Diode_SMD:D_SOD-123; manf# (none) -> MMSD4148T1G
- J4: manf# (none) -> BC-32677
- R1, R2, R3, R39, R4, R5, R6, R7: footprint (none) -> Resistor_SMD:R_0805_2012Metric
Connections:
- net +10V: now also Q1.2 (E)
- net +12V: now also Q1.3 (C)
- net at R6.2: now also Q1.1 (B)
Changed lines of the file:
@@
 F 2 "Connector_PinHeader_2.54mm:PinHeader_2x13_P2.54mm_Vertical" H 8300 4600 50  0001 C CNN
 F 3 "~" H 8300 4600 50  0001 C CNN
+F 4 "BC-32677" H 8300 4600 50  0001 C CNN "manf#"
 	1    8300 4600
 	1    0    0    -1
@@
 ECU_COOLANTTEMP
 $Comp
-L Device:D D3
-U 1 1 60492789
-P 7700 2550
-F 0 "D3" H 7700 2767 50  0000 C CNN
-F 1 "D" H 7700 2676 50  0000 C CNN
-F 2 "" H 7700 2550 50  0001 C CNN
-F 3 "~" H 7700 2550 50  0001 C CNN
-	1    7700 2550
-	1    0    0    -1
-$EndComp
-$Comp
 L Device:R R7
 U 1 1 60492E14
@@
 F 0 "R7" H 8170 2346 50  0000 L CNN
 F 1 "1k5" H 8170 2255 50  0000 L CNN
-F 2 "" V 8030 2300 50  0001 C CNN
+F 2 "Resistor_SMD:R_0805_2012Metric" V 8030 2300 50  0001 C CNN
 F 3 "~" H 8100 2300 50  0001 C CNN
 	1    8100 2300
@@
 F 0 "R4" V 2443 4950 50  0000 C CNN
 F 1 "240" V 2534 4950 50  0000 C CNN
-F 2 "" V 2580 4950 50  0001 C CNN
+F 2 "Resistor_SMD:R_0805_2012Metric" V 2580 4950 50  0001 C CNN
 F 3 "~" H 2650 4950 50  0001 C CNN
 	1    2650 4950
@@
 F 0 "R3" H 2420 4746 50  0000 L CNN
 F 1 "1k2" H 2420 4655 50  0000 L CNN
-F 2 "" V 2280 4700 50  0001 C CNN
+F 2 "Resistor_SMD:R_0805_2012Metric" V 2280 4700 50  0001 C CNN
 F 3 "~" H 2350 4700 50  0001 C CNN
 	1    2350 4700
@@
 P 2000 4950
 F 0 "D1" H 2000 5167 50  0000 C CNN
-F 1 "D" H 2000 5076 50  0000 C CNN
-F 2 "" H 2000 4950 50  0001 C CNN
+F 1 "MMSD4148T1G" H 2000 5076 50  0000 C CNN
+F 2 "Diode_SMD:D_SOD-123" H 2000 4950 50  0001 C CNN
 F 3 "~" H 2000 4950 50  0001 C CNN
+F 4 "MMSD4148T1G" H 2000 4950 50  0001 C CNN "manf#"
 	1    2000 4950
 	1    0    0    -1
@@
 F 0 "R2" V 1393 4950 50  0000 C CNN
 F 1 "2k2" V 1484 4950 50  0000 C CNN
-F 2 "" V 1530 4950 50  0001 C CNN
+F 2 "Resistor_SMD:R_0805_2012Metric" V 1530 4950 50  0001 C CNN
 F 3 "~" H 1600 4950 50  0001 C CNN
 	1    1600 4950
@@
 F 0 "R1" H 1320 4746 50  0000 L CNN
 F 1 "510" H 1320 4655 50  0000 L CNN
-F 2 "" V 1180 4700 50  0001 C CNN
+F 2 "Resistor_SMD:R_0805_2012Metric" V 1180 4700 50  0001 C CNN
 F 3 "~" H 1250 4700 50  0001 C CNN
 	1    1250 4700
@@
 F 0 "R5" H 4470 4596 50  0000 L CNN
 F 1 "680" H 4470 4505 50  0000 L CNN
-F 2 "" V 4330 4550 50  0001 C CNN
+F 2 "Resistor_SMD:R_0805_2012Metric" V 4330 4550 50  0001 C CNN
 F 3 "~" H 4400 4550 50  0001 C CNN
 	1    4400 4550
 	1    0    0    -1
-$EndComp
-$Comp
-L Device:D D2
-U 1 1 604BD1BA
-P 4400 5050
-F 0 "D2" V 4354 5130 50  0000 L CNN
-F 1 "D" V 4445 5130 50  0000 L CNN
-F 2 "" H 4400 5050 50  0001 C CNN
-F 3 "~" H 4400 5050 50  0001 C CNN
-	1    4400 5050
-	0    1    1    0
 $EndComp
 Wire Wire Line
@@
 F 0 "R6" V 4957 4850 50  0000 C CNN
 F 1 "150" V 4866 4850 50  0000 C CNN
-F 2 "" V 4680 4850 50  0001 C CNN
+F 2 "Resistor_SMD:R_0805_2012Metric" V 4680 4850 50  0001 C CNN
 F 3 "~" H 4750 4850 50  0001 C CNN
 	1    4750 4850
@@
 Wire Wire Line
 	4400 4850 4400 4900
-$Comp
-L Device:Q_NPN_CBE Q1
-U 1 1 604C3637
-P 5300 4450
-F 0 "Q1" V 5628 4450 50  0000 C CNN
-F 1 "BSX46" V 5537 4450 50  0000 C CNN
-F 2 "" H 5500 4550 50  0001 C CNN
-F 3 "~" H 5300 4450 50  0001 C CNN
-	1    5300 4450
-	0    -1   -1   0
-$EndComp
 Wire Wire Line
 	5100 4350 4400 4350
@@
 F 0 "R39" H 9820 2196 50  0000 L CNN
 F 1 "1k3" H 9820 2105 50  0000 L CNN
-F 2 "" V 9680 2150 50  0001 C CNN
+F 2 "Resistor_SMD:R_0805_2012Metric" V 9680 2150 50  0001 C CNN
 F 3 "~" H 9750 2150 50  0001 C CNN
 	1    9750 2150
@@
 	-1   0    0    -1
 $EndComp
+$Comp
+L Device:Q_NPN_BEC Q1
+U 1 1 605019F1
+P 5300 4450
+F 0 "Q1" V 5628 4450 50  0000 C CNN
+F 1 "BC817-40-TP" V 5537 4450 50  0000 C CNN
+F 2 "Package_TO_SOT_SMD:SOT-23" H 5500 4550 50  0001 C CNN
+F 3 "~" H 5300 4450 50  0001 C CNN
+F 4 "BC817-40-TP" V 5300 4450 50  0001 C CNN "manf#"
+	1    5300 4450
+	0    -1   -1   0
+$EndComp
+$Comp
+L Device:D D2
+U 1 1 60520E61
+P 4400 5050
+F 0 "D2" H 4400 5267 50  0000 C CNN
+F 1 "MMSD4148T1G" H 4400 5176 50  0000 C CNN
+F 2 "Diode_SMD:D_SOD-123" H 4400 5050 50  0001 C CNN
+F 3 "~" H 4400 5050 50  0001 C CNN
+F 4 "MMSD4148T1G" H 4400 5050 50  0001 C CNN "manf#"
+	1    4400 5050
+	0    1    1    0
+$EndComp
+$Comp
+L Device:D D3
+U 1 1 60521819
+P 7700 2550
+F 0 "D3" H 7700 2767 50  0000 C CNN
+F 1 "MMSD4148T1G" H 7700 2676 50  0000 C CNN
+F 2 "Diode_SMD:D_SOD-123" H 7700 2550 50  0001 C CNN
+F 3 "~" H 7700 2550 50  0001 C CNN
+F 4 "MMSD4148T1G" H 7700 2550 50  0001 C CNN "manf#"
+	1    7700 2550
+	1    0    0    -1
+$EndComp
 $EndSCHEMATC

Commit message: Laid out ECU outputs PCB. Generated manufacturing files.
Parts:
- J4: footprint Connector_PinHeader_2.54mm:PinHeader_2x13_P2.54mm_Vertical -> Connector_IDC:IDC-Header_2x13_P2.54mm_Vertical
Changed lines of the file:
@@
 F 0 "J4" H 8350 5417 50  0000 C CNN
 F 1 "ECU CONNECTOR" H 8350 5326 50  0000 C CNN
-F 2 "Connector_PinHeader_2.54mm:PinHeader_2x13_P2.54mm_Vertical" H 8300 4600 50  0001 C CNN
+F 2 "Connector_IDC:IDC-Header_2x13_P2.54mm_Vertical" H 8300 4600 50  0001 C CNN
 F 3 "~" H 8300 4600 50  0001 C CNN
 F 4 "BC-32677" H 8300 4600 50  0001 C CNN "manf#"
