File: DJet ECU Tester/PCB/DJetECUTester/DJetECUTester.sch (KiCad schematic (older format))
At the start: 26 parts, among them J1 ISP, J2 ECU, J4 BREAKOUT, J5 12V IN, J6 MPS, J8 INJECTORS, U1 ATmega328P, Y1 FA-238 16.0000MB-C3

Commit message: Renamed CSV to Start. Added PDF version of schematics.
Connections:
- net CSV renamed START
- net ECU_COLDSTARTRELAY renamed ECU_START
Changed lines of the file:
@@
 Sheet 1 7
 Title "D-Jetronic ECU Tester"
-Date "2021-03-15"
+Date "2021-03-20"
 Rev "1.0"
 Comp "(C) Britishideas 2021"
@@
 	8250 2450 7400 2450
 Text Label 8750 5450 0    50   ~ 0
-ECU_COLDSTARTRELAY
+ECU_START
 Text Label 8850 3050 0    50   ~ 0
-ECU_COLDSTARTRELAY
+ECU_START
 Wire Wire Line
 	8750 3050 8850 3050
@@
 Text Label 9200 1600 1    50   ~ 0
 ECU_INJGROUP4
-$Sheet
-S 1500 3850 900  300
-U 60469920
-F0 "CSV" 50
-F1 "CSV.sch" 50
-F2 "ECU_CSV" O R 2400 3950 50
-F3 "CSV" I L 1500 3950 50
-$EndSheet
 Text Label 2500 3950 0    50   ~ 0
-ECU_COLDSTARTRELAY
+ECU_START
 Wire Wire Line
 	2400 3950 2500 3950
@@
 	1500 3950 800  3950
 Text Label 800  3950 0    50   ~ 0
-CSV
+START
 Wire Wire Line
 	4550 2600 4750 2600
 Text Label 4750 2600 0    50   ~ 0
-CSV
+START
 $Comp
 L Device:Crystal_GND24 Y1
@@
 Wire Wire Line
 	5300 7050 5300 6850
+$Sheet
+S 1500 3850 900  300
+U 60469920
+F0 "Start" 50
+F1 "Start.sch" 50
+F2 "ECU_START" O R 2400 3950 50
+F3 "START" I L 1500 3950 50
+$EndSheet
 $EndSCHEMATC

Commit message: Working on version 1.1
Parts:
- removed J2: ECU, Connector_IDC:IDC-Header_2x13_P2.54mm_Vertical, symbol Connector_Generic:Conn_02x13_Odd_Even
- removed J8: INJECTORS, TerminalBlock_TE-Connectivity:TerminalBlock_TE_282834-8_1x08_P2.54mm_Horizontal, symbol Connector:Screw_Terminal_01x08
- removed JP1: RUN, Connector_PinHeader_2.54mm:PinHeader_1x02_P2.54mm_Vertical, symbol Connector_Generic:Conn_01x02
- added J10: ECU3, Britishideas:PhoenixContact_COMBICON_PT_7, symbol Connector:Screw_Terminal_01x07
- added J2: ECU1, Britishideas:PhoenixContact_COMBICON_PT_8, symbol Connector:Screw_Terminal_01x08
- added J8: INJECTORS, Britishideas:PhoenixContact_COMBICON_PT_5, symbol Connector:Screw_Terminal_01x05
- added J9: ECU2, Britishideas:PhoenixContact_COMBICON_PT_10, symbol Connector:Screw_Terminal_01x10
- J5: footprint TerminalBlock_TE-Connectivity:TerminalBlock_TE_282834-2_1x02_P2.54mm_Horizontal -> Britishideas:PhoenixContact_COMBICON_MKDSN_2; manf# 282834-2 -> 1729018
- J6: footprint TerminalBlock_TE-Connectivity:TerminalBlock_TE_282834-4_1x04_P2.54mm_Horizontal -> Britishideas:PhoenixContact_COMBICON_PT_4; manf# 282834-4 -> 1935792
Connections:
- net +12V: now also J5.2 (Pin_2), J2.1 (Pin_1), J2.2 (Pin_2); no longer J5.1 (Pin_1)
- net GND: now also J5.1 (Pin_1), J2.7 (Pin_7), J2.8 (Pin_8), J8.5 (Pin_5); no longer J5.2 (Pin_2)
- net MPS-10: now also J9.6 (Pin_6)
- net MPS-15: now also J9.9 (Pin_9)
- net MPS-7: now also J9.3 (Pin_3)
- net MPS-8: now also J9.4 (Pin_4)
- net ECU_AIRTEMP renamed ECU_AIRTEMP-1
- net ECU_AIRTEMP-1: now also J9.1 (Pin_1)
- net ECU_COOLANTTEMP renamed ECU_COOLANTTEMP-23
- net ECU_COOLANTTEMP-23: now also J10.6 (Pin_6)
- net ECU_DIAGGROUP13 renamed ECU_DIAGGROUP13-25
- net ECU_DIAGGROUP13-25: now also J10.7 (Pin_7)
- net ECU_FUELPUMPRELAY renamed ECU_FUELPUMPRELAY-19
- net ECU_FUELPUMPRELAY-19: now also J10.2 (Pin_2)
- net ECU_INJGROUP1 renamed ECU_INJGROUP1-3
- net ECU_INJGROUP1-3: now also J2.3 (Pin_3), J8.1 (Pin_1)
- net ECU_INJGROUP2 renamed ECU_INJGROUP2-4
- net ECU_INJGROUP2-4: now also J2.4 (Pin_4), J8.2 (Pin_2)
- net ECU_INJGROUP3 renamed ECU_INJGROUP3-5
- net ECU_INJGROUP3-5: now also J2.5 (Pin_5), J8.3 (Pin_3)
- net ECU_INJGROUP4 renamed ECU_INJGROUP4-6
- net ECU_INJGROUP4-6: now also J2.6 (Pin_6), J8.4 (Pin_4)
- net ECU_START renamed ECU_START-18
- net ECU_START-18: now also J10.1 (Pin_1)
- net ECU_TPSACCEL1 renamed ECU_TPSACCEL1-9
- net ECU_TPSACCEL1-9: now also J9.5 (Pin_5)
- net ECU_TPSACCEL2 renamed ECU_TPSACCEL2-20
- net ECU_TPSACCEL2-20: now also J10.3 (Pin_3)
- net ECU_TPSIDLE renamed ECU_TPSIDLE-17
- net ECU_TPSIDLE-17: now also J9.10 (Pin_10)
- net ECU_TPSWOT renamed ECU_TPSWOT-2
- net ECU_TPSWOT-2: now also J9.2 (Pin_2)
- net ECU_TRIGGERGROUP1 renamed ECU_TRIGGERGROUP1-21
- net ECU_TRIGGERGROUP1-21: now also J10.4 (Pin_4)
- net ECU_TRIGGERGROUP2 renamed ECU_TRIGGERGROUP2-13
- net ECU_TRIGGERGROUP2-13: now also J9.7 (Pin_7)
- net ECU_TRIGGERGROUP3 renamed ECU_TRIGGERGROUP3-22
- net ECU_TRIGGERGROUP3-22: now also J10.5 (Pin_5)
- net ECU_TRIGGERGROUP4 renamed ECU_TRIGGERGROUP4-14
- net ECU_TRIGGERGROUP4-14: now also J9.8 (Pin_8)
- no-connect marks 4 -> 3
Other:
- note added: "Min 3A connector"
- note removed: "Current draw on pin 24 could be as high as 6A. 20 AWG wiring needed"
- moved on the sheet: D1, J6, R4, R5
