File: DJet ECU Tester/PCB/DJetECUTester/Temperature.sch (KiCad schematic (older format))
At the start: 10 parts, among them U4 MCP41HV51-502E-ST, U5 MCP41HV51-502E-ST

Commit message: Working on ECU tester and ECU outputs board.
Parts:
- U4: footprint (none) -> Package_SO:TSSOP-14_4.4x5mm_P0.65mm; manf# (none) -> MCP41HV51-502E/ST
- U5: footprint (none) -> Package_SO:TSSOP-14_4.4x5mm_P0.65mm; manf# (none) -> MCP41HV51-502E-ST
Changed lines of the file:
@@
 $Descr A4 11693 8268
 encoding utf-8
-Sheet 4 6
+Sheet 4 7
 Title "D-Jetronic ECU Tester"
-Date "2021-03-04"
+Date "2021-03-08"
 Rev "1.0"
 Comp "(C) Britishideas 2021"
@@
 F 0 "U4" H 5550 4015 50  0000 C CNN
 F 1 "MCP41HV51-502E-ST" H 5550 3924 50  0000 C CNN
-F 2 "" H 5250 3050 50  0001 C CNN
+F 2 "Package_SO:TSSOP-14_4.4x5mm_P0.65mm" H 5250 3050 50  0001 C CNN
 F 3 "" H 5250 3050 50  0001 C CNN
+F 4 "" H 5250 3050 50  0001 C CNN "Field4"
+F 5 "MCP41HV51-502E/ST" H 5250 3050 50  0001 C CNN "manf#"
 	1    5250 3050
 	1    0    0    -1
@@
 F 0 "U5" H 5550 6315 50  0000 C CNN
 F 1 "MCP41HV51-502E-ST" H 5550 6224 50  0000 C CNN
-F 2 "" H 5250 5350 50  0001 C CNN
+F 2 "Package_SO:TSSOP-14_4.4x5mm_P0.65mm" H 5250 5350 50  0001 C CNN
 F 3 "" H 5250 5350 50  0001 C CNN
+F 4 "MCP41HV51-502E-ST" H 5250 5350 50  0001 C CNN "manf#"
 	1    5250 5350
 	1    0    0    -1

Commit message: Started work on PCB.
Parts:
- TP1, TP2, TP3, TP4: footprint TestPoint:TestPoint_Pad_D4.0mm -> TestPoint:TestPoint_Pad_D2.0mm
Changed lines of the file:
@@
 F 0 "TP1" H 6408 2568 50  0000 L CNN
 F 1 "TestPoint" H 6408 2477 50  0000 L CNN
-F 2 "TestPoint:TestPoint_Pad_D4.0mm" H 6550 2450 50  0001 C CNN
+F 2 "TestPoint:TestPoint_Pad_D2.0mm" H 6550 2450 50  0001 C CNN
 F 3 "~" H 6550 2450 50  0001 C CNN
 	1    6350 2450
@@
 F 0 "TP2" H 6292 2676 50  0000 R CNN
 F 1 "TestPoint" H 6292 2767 50  0000 R CNN
-F 2 "TestPoint:TestPoint_Pad_D4.0mm" H 6550 2650 50  0001 C CNN
+F 2 "TestPoint:TestPoint_Pad_D2.0mm" H 6550 2650 50  0001 C CNN
 F 3 "~" H 6550 2650 50  0001 C CNN
 	1    6350 2650
@@
 F 0 "TP3" H 6408 4868 50  0000 L CNN
 F 1 "TestPoint" H 6408 4777 50  0000 L CNN
-F 2 "TestPoint:TestPoint_Pad_D4.0mm" H 6550 4750 50  0001 C CNN
+F 2 "TestPoint:TestPoint_Pad_D2.0mm" H 6550 4750 50  0001 C CNN
 F 3 "~" H 6550 4750 50  0001 C CNN
 	1    6350 4750
@@
 F 0 "TP4" H 6292 4976 50  0000 R CNN
 F 1 "TestPoint" H 6292 5067 50  0000 R CNN
-F 2 "TestPoint:TestPoint_Pad_D4.0mm" H 6550 4950 50  0001 C CNN
+F 2 "TestPoint:TestPoint_Pad_D2.0mm" H 6550 4950 50  0001 C CNN
 F 3 "~" H 6550 4950 50  0001 C CNN
 	1    6350 4950

Commit message: Working on PCB layout. Changed CSV circuit from optocoupler to transistors. Added decoupling caps for digital pots.
Parts:
- added C14, C15, C16, C17: 100nF, Capacitor_SMD:C_0805_2012Metric, symbol Device:C
Connections:
- net +12V: now also C16.1, C17.1
- net +5V: now also C14.1, C15.1
- net GND: now also C14.2, C15.2, C16.2, C17.2
Other:
- moved on the sheet: JP2, JP3, R15, R16, TP1, TP2, TP3, TP4, U4, U5

Commit message: Updated manufacturer part numbers. Working on ECU outputs tester board.
Parts:
- U5: manf# MCP41HV51-502E-ST -> MCP41HV51-502E/ST
Changed lines of the file:
@@
 F 2 "Package_SO:TSSOP-14_4.4x5mm_P0.65mm" H 6050 5450 50  0001 C CNN
 F 3 "" H 6050 5450 50  0001 C CNN
-F 4 "MCP41HV51-502E-ST" H 6050 5450 50  0001 C CNN "manf#"
+F 4 "MCP41HV51-502E/ST" H 6050 5450 50  0001 C CNN "manf#"
 	1    6050 5450
 	1    0    0    -1
