File: DJet ECU Tester/PCB/DJetECUTester/USBandPower.sch (KiCad schematic (older format))
At the start: 16 parts, among them J3 USB_B_Mini, U2 LM2596S-5, U3 FT232RL

Commit message: Working on ECU tester and ECU outputs board.
Parts:
- D4: footprint Britishideas:SMP_DO-220AA -> Britishideas:SOD-123
- FB1: footprint (none) -> Resistor_SMD:R_0805_2012Metric; manf# (none) -> MI0805K400R-10
- L1: footprint Britishideas:Chilisin_Power_Inductor_AWVS_808040 -> Britishideas:Wurth-WE-LQS-Inductor
Changed lines of the file:
@@
 $Descr A4 11693 8268
 encoding utf-8
-Sheet 2 6
+Sheet 2 7
 Title "D-Jetronic ECU Tester"
-Date "2021-03-04"
+Date "2021-03-08"
 Rev "1.0"
 Comp "(C) Britishideas 2021"
@@
 F 0 "L1" V 4900 5850 50  0000 C CNN
 F 1 "33uH" V 5049 5850 50  0000 C CNN
-F 2 "Britishideas:Chilisin_Power_Inductor_AWVS_808040" H 4950 5850 50  0001 C CNN
+F 2 "Britishideas:Wurth-WE-LQS-Inductor" H 4950 5850 50  0001 C CNN
 F 3 "~" H 4950 5850 50  0001 C CNN
 	1    4950 5850
@@
 F 0 "D4" H 9000 3817 50  0000 C CNN
 F 1 "MBR0520LT1G" H 9000 3726 50  0000 C CNN
-F 2 "Britishideas:SMP_DO-220AA" H 9000 3600 50  0001 C CNN
+F 2 "Britishideas:SOD-123" H 9000 3600 50  0001 C CNN
 F 3 "~" H 9000 3600 50  0001 C CNN
 	1    9000 3600
@@
 F 0 "FB1" H 3200 2500 50  0000 R CNN
 F 1 "MI0805K400R-10" H 3750 2600 50  0000 R CNN
-F 2 "" V 2830 2550 50  0001 C CNN
+F 2 "Resistor_SMD:R_0805_2012Metric" V 2830 2550 50  0001 C CNN
 F 3 "~" H 2900 2550 50  0001 C CNN
+F 4 "MI0805K400R-10" H 2900 2550 50  0001 C CNN "manf#"
 	1    2900 2550
 	-1   0    0    1

Commit message: Adding 3D models.
Parts:
- L1: manf# (none) -> 74404063330
Changed lines of the file:
@@
 F 2 "Britishideas:Wurth-WE-LQS-Inductor" H 4950 5850 50  0001 C CNN
 F 3 "~" H 4950 5850 50  0001 C CNN
+F 4 "74404063330" V 4950 5850 50  0001 C CNN "manf#"
 	1    4950 5850
 	0    -1   -1   0

Commit message: Updated manufacturer part numbers. Working on ECU outputs tester board.
Parts:
- D2: manf# (none) -> B360A-13-F
- D4: manf# (none) -> MBR0520LT1G
- J3: manf# (none) -> 65100516121
- U2: manf# (none) -> LM2596S-5.0/NOPB
- U3: manf# (none) -> FT232RL-REEL
Changed lines of the file:
@@
 F 2 "Package_TO_SOT_SMD:TO-263-5_TabPin3" H 4050 5500 50  0001 L CIN
 F 3 "http://www.ti.com/lit/ds/symlink/lm2596.pdf" H 4000 5750 50  0001 C CNN
+F 4 "LM2596S-5.0/NOPB" H 4000 5750 50  0001 C CNN "manf#"
 	1    4000 5750
 	1    0    0    -1
@@
 F 2 "Diode_SMD:D_SMA" H 4700 6000 50  0001 C CNN
 F 3 "~" H 4700 6000 50  0001 C CNN
+F 4 "B360A-13-F" V 4700 6000 50  0001 C CNN "manf#"
 	1    4700 6000
 	0    1    1    0
@@
 F 2 "Britishideas:SOD-123" H 9000 3600 50  0001 C CNN
 F 3 "~" H 9000 3600 50  0001 C CNN
+F 4 "MBR0520LT1G" H 9000 3600 50  0001 C CNN "manf#"
 	1    9000 3600
 	1    0    0    -1
@@
 F 2 "Package_SO:SSOP-28_5.3x10.2mm_P0.65mm" H 5650 2150 50  0001 C CNN
 F 3 "https://www.ftdichip.com/Support/Documents/DataSheets/ICs/DS_FT232R.pdf" H 4550 3050 50  0001 C CNN
+F 4 "FT232RL-REEL" H 4550 3050 50  0001 C CNN "manf#"
 	1    4550 3050
 	1    0    0    -1
@@
 F 2 "Connector_USB:USB_Mini-B_Wuerth_65100516121_Horizontal" H 2600 3150 50  0001 C CNN
 F 3 "~" H 2600 3150 50  0001 C CNN
+F 4 "65100516121" H 2450 3200 50  0001 C CNN "manf#"
 	1    2450 3200
 	1    0    0    -1
