File: CloneECU/PCB/CloneECU.sch (KiCad schematic (older format))
At the start: 1 part

Commit message: Removed components external to the ECU. Changed text blocks. Passes the electrical DRC.
Connections:
- net E10-MPS renamed Int-6
Changed lines of the file:
@@
 encoding utf-8
 Sheet 1 6
-Title "Bosch D-Jetronic ECU 0 280 002 005"
-Date "2020-08-09"
-Rev "1.05"
-Comp "Mercedes-Benz"
+Title "R/C107 D-Jetronic ECU Clone"
+Date "2021-07-23"
+Rev "1.00"
+Comp ""
 Comment1 "M117.982 Engine"
-Comment2 "Bosch Order # 0 280 002 005"
-Comment3 "Mercedes-Benz Part # A 000 545 26 32"
+Comment2 "Clone of Bosch # 0 280 002 005"
+Comment3 "Clone of Mercedes-Benz Part # A 000 545 26 32"
 Comment4 "Input / Output & Interior Connections"
 $EndDescr
@@
 Text GLabel 5900 4200 2    50   Input ~ 0
 E7-MPS
-Text GLabel 5900 4800 2    50   Input ~ 0
-E10-MPS
 Text GLabel 5900 5400 2    50   Input ~ 0
 E13-PG
@@
 Text Notes 6400 5050 0    50   ~ 0
 ECU Ground (M5 on intake manifold)
-Text GLabel 5900 5200 2    50   UnSpc ~ 0
-E12-GND
 Text Notes 6400 5250 0    50   ~ 0
 TPS & PG Ground (internal tie to E11)
@@
 Text Notes 12650 4450 0    50   ~ 0
 Coolant Temp Bias
-Text GLabel 12100 7600 2    50   BiDi ~ 0
-Int-6
 Text GLabel 12100 7400 2    50   BiDi ~ 0
 Int-5
@@
 Wire Wire Line
 	5750 8250 5750 4800
+Text GLabel 12100 7600 2    50   BiDi ~ 0
+Int-6
+Text Label 5900 4800 0    50   ~ 0
+E10-MPS
+Text Label 5900 5200 0    50   ~ 0
+E12-GND
 $EndSCHEMATC
